File: Karnix_ASB-254-v1.0/Ethernet.kicad_sch (KiCad schematic)
At the start: 55 parts, among them U8 LAN8710AI

Commit message: Fix power supply, use +3V3 rail instead
Connections:
- net +3V3_ETH: no longer C42.1, C43.1, L3.2, R82.1, R83.1, R84.1, R85.1, R86.1, R87.1, R88.1, U8.12 (VDDIO)
- new net +3V3: C42.1, C43.1, L3.2, R82.1, R83.1, R84.1, R85.1, R86.1, R87.1, R88.1, U8.12 (VDDIO)
Changed lines of the file:
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@@
-    )
-  )
-  (symbol (lib_id "Fabmicro:+3V3_ETH") (at 202.565 50.8 0) (unit 1)
-    (in_bom yes) (on_board yes) (dnp no)
-    (property "Reference" "#PWR0108" (at 202.565 54.61 0)
-      (effects (font (size 1.27 1.27)) hide)
-    )
-    (property "Value" "+3V3_ETH" (at 202.565 46.99 0)
-      (effects (font (size 1.27 1.27)))
-    )
-    (property "Footprint" "" (at 202.565 50.8 0)
-      (effects (font (size 1.27 1.27)) hide)
-    )
-    (property "Datasheet" "" (at 202.565 50.8 0)
-      (effects (font (size 1.27 1.27)) hide)
-    )
-    (pin "1")
-    (instances
-      (project "Karnix_ASB"
-        (path "/fe37e245-9527-4c72-91fc-09b617a42f73/00000000-0000-0000-0000-0000602e11fa"
-          (reference "#PWR0108") (unit 1)
-        )
-      )
     )
   )
@@
         (path "/fe37e245-9527-4c72-91fc-09b617a42f73/00000000-0000-0000-0000-0000602e11fa"
           (reference "R76") (unit 1)
-        )
-      )
-    )
-  )
-  (symbol (lib_id "Fabmicro:+3V3_ETH") (at 151.765 132.08 0) (unit 1)
-    (in_bom yes) (on_board yes) (dnp no)
-    (property "Reference" "#PWR0117" (at 151.765 135.89 0)
-      (effects (font (size 1.27 1.27)) hide)
-    )
-    (property "Value" "+3V3_ETH" (at 152.146 127.6858 0)
-      (effects (font (size 1.27 1.27)))
-    )
-    (property "Footprint" "" (at 151.765 132.08 0)
-      (effects (font (size 1.27 1.27)) hide)
-    )
-    (property "Datasheet" "" (at 151.765 132.08 0)
-      (effects (font (size 1.27 1.27)) hide)
-    )
-    (pin "1")
-    (instances
-      (project "Karnix_ASB"
-        (path "/fe37e245-9527-4c72-91fc-09b617a42f73/00000000-0000-0000-0000-0000602e11fa"
-          (reference "#PWR0117") (unit 1)
         )
       )
@@
         (path "/fe37e245-9527-4c72-91fc-09b617a42f73/00000000-0000-0000-0000-0000602e11fa"
           (reference "R82") (unit 1)
-        )
-      )
-    )
-  )
-  (symbol (lib_id "Fabmicro:+3V3_ETH") (at 45.085 132.08 0) (unit 1)
-    (in_bom yes) (on_board yes) (dnp no)
-    (property "Reference" "#PWR0116" (at 45.085 135.89 0)
-      (effects (font (size 1.27 1.27)) hide)
-    )
-    (property "Value" "+3V3_ETH" (at 45.085 128.27 0)
-      (effects (font (size 1.27 1.27)))
-    )
-    (property "Footprint" "" (at 45.085 132.08 0)
-      (effects (font (size 1.27 1.27)) hide)
-    )
-    (property "Datasheet" "" (at 45.085 132.08 0)
-      (effects (font (size 1.27 1.27)) hide)
-    )
-    (pin "1")
-    (instances
-      (project "Karnix_ASB"
-        (path "/fe37e245-9527-4c72-91fc-09b617a42f73/00000000-0000-0000-0000-0000602e11fa"
-          (reference "#PWR0116") (unit 1)
         )
       )
@@
         )
       )
+    )
+  )
+  (symbol (lib_id "Fabmicro:+3V3") (at 151.765 132.08 0) (unit 1)
+    (in_bom yes) (on_board yes) (dnp no) (fields_autoplaced)
+    (property "Reference" "#PWR050" (at 151.765 135.89 0)
+      (effects (font (size 1.27 1.27)) hide)
+    )
+    (property "Value" "+3V3" (at 151.765 128.5129 0)
+      (effects (font (size 1.27 1.27)))
+    )
+    (property "Footprint" "" (at 151.765 132.08 0)
+      (effects (font (size 1.27 1.27)) hide)
+    )
+    (property "Datasheet" "" (at 151.765 132.08 0)
+      (effects (font (size 1.27 1.27)) hide)
+    )
+    (pin "1")
+    (instances
+      (project "Karnix_ASB"
+        (path "/fe37e245-9527-4c72-91fc-09b617a42f73/00000000-0000-0000-0000-0000602e0fd3"
+          (reference "#PWR050") (unit 1)
+        )
+        (path "/fe37e245-9527-4c72-91fc-09b617a42f73/00000000-0000-0000-0000-0000602e11fa"
+          (reference "#PWR0116") (unit 1)
+        )
+      )
+    )
+  )
+  (symbol (lib_id "Fabmicro:+3V3") (at 45.085 132.08 0) (unit 1)
+    (in_bom yes) (on_board yes) (dnp no) (fields_autoplaced)
+    (property "Reference" "#PWR050" (at 45.085 135.89 0)
+      (effects (font (size 1.27 1.27)) hide)
+    )
+    (property "Value" "+3V3" (at 45.085 128.5129 0)
+      (effects (font (size 1.27 1.27)))
+    )
+    (property "Footprint" "" (at 45.085 132.08 0)
+      (effects (font (size 1.27 1.27)) hide)
+    )
+    (property "Datasheet" "" (at 45.085 132.08 0)
+      (effects (font (size 1.27 1.27)) hide)
+    )
+    (pin "1")
+    (instances
+      (project "Karnix_ASB"
+        (path "/fe37e245-9527-4c72-91fc-09b617a42f73/00000000-0000-0000-0000-0000602e0fd3"
+          (reference "#PWR050") (unit 1)
+        )
+        (path "/fe37e245-9527-4c72-91fc-09b617a42f73/00000000-0000-0000-0000-0000602e11fa"
+          (reference "#PWR095") (unit 1)
+        )
+      )
+    )
+  )
+  (symbol (lib_id "Fabmicro:+3V3") (at 202.565 50.8 0) (unit 1)
+    (in_bom yes) (on_board yes) (dnp no) (fields_autoplaced)
+    (property "Reference" "#PWR050" (at 202.565 54.61 0)
+      (effects (font (size 1.27 1.27)) hide)
+    )
+    (property "Value" "+3V3" (at 202.565 47.2329 0)
+      (effects (font (size 1.27 1.27)))
+    )
+    (property "Footprint" "" (at 202.565 50.8 0)
+      (effects (font (size 1.27 1.27)) hide)
+    )
+    (property "Datasheet" "" (at 202.565 50.8 0)
+      (effects (font (size 1.27 1.27)) hide)
+    )
+    (pin "1")
+    (instances
+      (project "Karnix_ASB"
+        (path "/fe37e245-9527-4c72-91fc-09b617a42f73/00000000-0000-0000-0000-0000602e0fd3"
+          (reference "#PWR050") (unit 1)
+        )
+        (path "/fe37e245-9527-4c72-91fc-09b617a42f73/00000000-0000-0000-0000-0000602e11fa"
+          (reference "#PWR0108") (unit 1)
+        )
+      )

Commit message: Add passive PoE feature
Parts:
- added D8: STPS2L40AF, Fabmicro:D_SMA_FLAT, symbol Fabmicro:Diode
Connections:
- net +3V3: now also R66.1, R67.1
- net +3V3_ETH: no longer R66.1, R67.1
- net +12V0: no longer names the net of XS4.4, XS4.5
- net +12V0: now also D8.2 (A)
- new net DCIN: D8.1 (K)
Other:
- note added: "Passove PoE"
Changed lines of the file:
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@@
   (junction (at 95.885 162.56) (diameter 0) (color 0 0 0 0)
   )
-  (junction (at 45.085 210.82) (diameter 0) (color 0 0 0 0)
-  )
   (junction (at 45.085 220.98) (diameter 0) (color 0 0 0 0)
   )
@@
   (junction (at 207.645 210.82) (diameter 0) (color 0 0 0 0)
   )
+  (junction (at 45.085 210.82) (diameter 0) (color 0 0 0 0)
+  )
   (junction (at 151.765 149.86) (diameter 0) (color 0 0 0 0)
   )
@@
     (stroke (width 0) (type default))
   )
-  (wire (pts (xy 45.085 210.82) (xy 45.085 195.58))
-    (stroke (width 0) (type default))
-  )
   (wire (pts (xy 222.885 71.12) (xy 233.045 71.12))
     (stroke (width 0) (type default))
@@
     (stroke (width 0) (type default))
   )
+  (wire (pts (xy 47.68 197.5) (xy 45.1 197.5))
+    (stroke (width 0) (type default))
+  )
   (wire (pts (xy 78.105 256.54) (xy 78.105 259.08))
     (stroke (width 0) (type default))
@@
     (stroke (width 0) (type default))
   )
-  (wire (pts (xy 42.545 210.82) (xy 45.085 210.82))
-    (stroke (width 0) (type default))
-  )
   (wire (pts (xy 106.045 147.32) (xy 106.045 165.1))
     (stroke (width 0) (type default))
@@
     (stroke (width 0) (type default))
   )
+  (wire (pts (xy 45.1 197.5) (xy 45.1 210.82))
+    (stroke (width 0) (type default))
+  )
   (wire (pts (xy 65.405 182.88) (xy 65.405 180.34))
     (stroke (width 0) (type default))
@@
     (stroke (width 0) (type default))
   )
+  (wire (pts (xy 45.1 210.82) (xy 45.085 210.82))
+    (stroke (width 0) (type default))
+  )
   (wire (pts (xy 55.245 266.7) (xy 52.705 266.7))
     (stroke (width 0) (type default))
@@
     (stroke (width 0) (type default))
   )
+  (wire (pts (xy 42.545 210.82) (xy 45.085 210.82))
+    (stroke (width 0) (type default))
+  )
   (wire (pts (xy 227.965 187.96) (xy 227.965 185.42))
     (stroke (width 0) (type default))
@@
     (effects (font (size 1.27 1.27)) (justify left bottom))
   )
+  (text "Passove PoE" (at 46 213 0)
+    (effects (font (size 1.27 1.27)) (justify left bottom))
+  )
   (text "PA11/MDC_LAN8710" (at 50.165 96.52 0)
     (effects (font (size 1.27 1.27)) (justify left bottom))
@@
     )
   )
-  (symbol (lib_id "Fabmicro:+3V3_ETH") (at 95.885 38.1 0) (unit 1)
-    (in_bom yes) (on_board yes) (dnp no)
-    (property "Reference" "#PWR0107" (at 95.885 41.91 0)
-      (effects (font (size 1.27 1.27)) hide)
-    )
-    (property "Value" "+3V3_ETH" (at 95.885 34.29 0)
-      (effects (font (size 1.27 1.27)))
-    )
-    (property "Footprint" "" (at 95.885 38.1 0)
-      (effects (font (size 1.27 1.27)) hide)
-    )
-    (property "Datasheet" "" (at 95.885 38.1 0)
-      (effects (font (size 1.27 1.27)) hide)
-    )
-    (pin "1")
-    (instances
-      (project "Karnix_ASB"
-        (path "/fe37e245-9527-4c72-91fc-09b617a42f73/00000000-0000-0000-0000-0000602e11fa"
-          (reference "#PWR0107") (unit 1)
-        )
-      )
-    )
-  )
   (symbol (lib_id "Fabmicro:CapacitorUnpolarized") (at 222.885 83.82 270) (unit 1)
     (in_bom yes) (on_board yes) (dnp no)
@@
     )
   )
-  (symbol (lib_id "Fabmicro:+12V0") (at 45.085 195.58 0) (unit 1)
-    (in_bom yes) (on_board yes) (dnp no)
-    (property "Reference" "#PWR0128" (at 45.085 199.39 0)
-      (effects (font (size 1.27 1.27)) hide)
-    )
-    (property "Value" "+12V0" (at 45.085 191.77 0)
-      (effects (font (size 1.27 1.27)))
-    )
-    (property "Footprint" "" (at 45.085 195.58 0)
-      (effects (font (size 1.27 1.27)) hide)
-    )
-    (property "Datasheet" "" (at 45.085 195.58 0)
-      (effects (font (size 1.27 1.27)) hide)
-    )
-    (pin "1")
-    (instances
-      (project "Karnix_ASB"
-        (path "/fe37e245-9527-4c72-91fc-09b617a42f73/00000000-0000-0000-0000-0000602e11fa"
-          (reference "#PWR0128") (unit 1)
-        )
-      )
-    )
-  )
   (symbol (lib_id "Fabmicro:Resistor") (at 95.885 175.26 90) (mirror x) (unit 1)
     (in_bom yes) (on_board yes) (dnp no)
@@
     )
   )
+  (symbol (lib_id "Fabmicro:Diode") (at 55.3 197.5 180) (unit 1)
+    (in_bom yes) (on_board yes) (dnp no)
+    (property "Reference" "D8" (at 53.395 192.42 90)
+      (effects (font (size 1.27 1.27)) (justify right))
+    )
+    (property "Value" "STPS2L40AF" (at 47.4 200.2 0)
+      (effects (font (size 1.27 1.27)) (justify right))
+    )
+    (property "Footprint" "Fabmicro:D_SMA_FLAT" (at 51.49 197.5 0)
+      (effects (font (size 1.27 1.27)) hide)
+    )
+    (property "Datasheet" "~" (at 51.49 197.5 0)
+      (effects (font (size 1.27 1.27)) hide)
+    )
+    (property "Mfr. Part Number" "STPS2L40AF" (at 55.3 197.5 0)
+      (effects (font (size 1.27 1.27)) hide)
+    )
+    (property "Supplier" "Elitan" (at 55.3 197.5 0)
+      (effects (font (size 1.27 1.27)) hide)
+    )
+    (pin "1")
+    (pin "2")
+    (instances
+      (project "Karnix_ASB"
+        (path "/fe37e245-9527-4c72-91fc-09b617a42f73/00000000-0000-0000-0000-0000602e0fd3"
+          (reference "D8") (unit 1)
+        )
+        (path "/fe37e245-9527-4c72-91fc-09b617a42f73/00000000-0000-0000-0000-0000602e11fa"
+          (reference "D23") (unit 1)
+        )
+      )
+    )
+  )
   (symbol (lib_id "Fabmicro:+3V3") (at 45.085 132.08 0) (unit 1)
     (in_bom yes) (on_board yes) (dnp no) (fields_autoplaced)
@@
         )
       )
+    )
+  )
+  (symbol (lib_id "Fabmicro:+3V3") (at 95.885 38.1 0) (unit 1)
+    (in_bom yes) (on_board yes) (dnp no) (fields_autoplaced)
+    (property "Reference" "#PWR050" (at 95.885 41.91 0)
+      (effects (font (size 1.27 1.27)) hide)
+    )
+    (property "Value" "+3V3" (at 95.885 34.5329 0)
+      (effects (font (size 1.27 1.27)))
+    )
+    (property "Footprint" "" (at 95.885 38.1 0)
+      (effects (font (size 1.27 1.27)) hide)
+    )
+    (property "Datasheet" "" (at 95.885 38.1 0)
+      (effects (font (size 1.27 1.27)) hide)
+    )
+    (pin "1")
+    (instances
+      (project "Karnix_ASB"
+        (path "/fe37e245-9527-4c72-91fc-09b617a42f73/00000000-0000-0000-0000-0000602e0fd3"
+          (reference "#PWR050") (unit 1)
+        )
+        (path "/fe37e245-9527-4c72-91fc-09b617a42f73/00000000-0000-0000-0000-0000602e11fa"
+          (reference "#PWR0107") (unit 1)
+        )
+      )
+    )
+  )
+  (symbol (lib_id "Fabmicro:DCIN") (at 55.3 197.5 270) (unit 1)
+    (in_bom yes) (on_board yes) (dnp no)
+    (property "Reference" "#PWR03" (at 51.49 197.5 0)
+      (effects (font (size 1.27 1.27)) hide)
+    )
+    (property "Value" "DCIN" (at 58.5 197.5 90)
+      (effects (font (size 1.27 1.27)) (justify left))
+    )
+    (property "Footprint" "" (at 55.3 197.5 0)
+      (effects (font (size 1.27 1.27)) hide)
+    )
+    (property "Datasheet" "" (at 55.3 197.5 0)
+      (effects (font (size 1.27 1.27)) hide)
+    )
+    (pin "1")
+    (instances
+      (project "Karnix_ASB"
+        (path "/fe37e245-9527-4c72-91fc-09b617a42f73"
+          (reference "#PWR03") (unit 1)
+        )
+        (path "/fe37e245-9527-4c72-91fc-09b617a42f73/00000000-0000-0000-0000-0000602e0fd3"
+          (reference "#PWR022") (unit 1)
+        )
+        (path "/fe37e245-9527-4c72-91fc-09b617a42f73/00000000-0000-0000-0000-0000602e11fa"
+          (reference "#PWR0128") (unit 1)
+        )
+      )
