File: Karnix_ASB-254-v1.0/Ethernet.kicad_sch (KiCad schematic)
At the start: 56 parts, among them U8 LAN8710AI

Commit message: Optimize component base
Parts:
- C42, C46: value 22uF/25V -> 22uF/10V; Mfr. Part Number GRT21BR61E226ME13L -> TCC0805X5R226M100FT
- L3: value BLM18PG331SN1D -> 330R/1.2A
Changed lines of the file:
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@@
   (title_block
     (title "ПИР СЦХ-254 \"Карно\"\n(Karnix ASB-254)")
-    (date "2023-10-20")
+    (date "2023-10-21")
     (rev "V1.0")
     (company "ООО \"Фабмикро\"")
@@
       (effects (font (size 1.27 1.27)) (justify left))
     )
-    (property "Value" "22uF/25V" (at 203.835 63.5 90)
+    (property "Value" "22uF/10V" (at 203.835 63.5 90)
       (effects (font (size 1.27 1.27)) (justify left))
     )
@@
       (effects (font (size 1.27 1.27)) hide)
     )
-    (property "Mfr. Part Number" "GRT21BR61E226ME13L" (at 202.565 60.96 0)
+    (property "Mfr. Part Number" "TCC0805X5R226M100FT" (at 202.565 60.96 0)
       (effects (font (size 1.27 1.27)) hide)
     )
@@
       (effects (font (size 1.27 1.27)))
     )
-    (property "Value" "BLM18PG331SN1D" (at 222.885 58.42 0)
+    (property "Value" "330R/1.2A" (at 222.885 58.42 0)
       (effects (font (size 1.27 1.27)))
     )
@@
       (effects (font (size 1.27 1.27)) (justify left))
     )
-    (property "Value" "22uF/25V" (at 224.155 86.36 90)
+    (property "Value" "22uF/10V" (at 224.155 86.36 90)
       (effects (font (size 1.27 1.27)) (justify left))
     )
@@
       (effects (font (size 1.27 1.27)) hide)
     )
-    (property "Mfr. Part Number" "GRT21BR61E226ME13L" (at 222.885 83.82 0)
-      (effects (font (size 1.27 1.27)) hide)
-    )
+    (property "Mfr. Part Number" "TCC0805X5R226M100FT" (at 222.885 83.82 0)
+      (effects (font (size 1.27 1.27)) hide)
+    )
