File: Karnix_ASB-254-v1.0/RS485.kicad_sch (KiCad schematic)
At the start: 11 parts, among them U9 MAX487ECSA+

Commit message: Fix power rail to RS485 transciever
Connections:
- net +5V0_IN renamed +5V
Changed lines of the file:
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@@
+    )
+  )
+  (symbol (lib_id "power:+5V") (at 162.306 103.251 0) (unit 1)
+    (in_bom yes) (on_board yes) (dnp no) (fields_autoplaced)
+    (property "Reference" "#PWR020" (at 162.306 107.061 0)
+      (effects (font (size 1.27 1.27)) hide)
+    )
+    (property "Value" "+5V" (at 162.306 99.6839 0)
+      (effects (font (size 1.27 1.27)))
+    )
+    (property "Footprint" "" (at 162.306 103.251 0)
+      (effects (font (size 1.27 1.27)) hide)
+    )
+    (property "Datasheet" "" (at 162.306 103.251 0)
+      (effects (font (size 1.27 1.27)) hide)
+    )
+    (pin "1")
+    (instances
+      (project "Karnix_ASB"
+        (path "/fe37e245-9527-4c72-91fc-09b617a42f73/00000000-0000-0000-0000-0000602e0fd3"
+          (reference "#PWR020") (unit 1)
+        )
+        (path "/fe37e245-9527-4c72-91fc-09b617a42f73/837bd409-d02c-43f6-9938-fa1825fbf100"
+          (reference "#PWR0220") (unit 1)
+        )
+      )
     )
   )
@@
         )
       )
-    )
-  )
-  (symbol (lib_id "Fabmicro:+5V0_IN") (at 162.306 103.251 0) (mirror y) (unit 1)
-    (in_bom yes) (on_board yes) (dnp no)
-    (property "Reference" "#PWR0128" (at 162.306 107.061 0)
-      (effects (font (size 1.27 1.27)) hide)
-    )
-    (property "Value" "+5V0_IN" (at 162.306 99.441 0)
-      (effects (font (size 1.27 1.27)))
-    )
-    (property "Footprint" "" (at 162.306 103.251 0)
-      (effects (font (size 1.27 1.27)) hide)
-    )
-    (property "Datasheet" "" (at 162.306 103.251 0)
-      (effects (font (size 1.27 1.27)) hide)
-    )
-    (pin "1")
-    (instances
-      (project "Karnix_ASB"
-        (path "/fe37e245-9527-4c72-91fc-09b617a42f73/00000000-0000-0000-0000-0000602e11fa"
-          (reference "#PWR0128") (unit 1)
-        )
-        (path "/fe37e245-9527-4c72-91fc-09b617a42f73/00000000-0000-0000-0000-0000602e0fd3"
-          (reference "#PWR?") (unit 1)
-        )
-        (path "/fe37e245-9527-4c72-91fc-09b617a42f73/837bd409-d02c-43f6-9938-fa1825fbf100"
-          (reference "#PWR0137") (unit 1)
-        )
-      )
