File: Karnix_ASB-254-v1.0/HDMI.kicad_sch (KiCad schematic)
At the start: 41 parts, among them J3 HDMI_A_1.4, Q2 DMN3730, Q3 DMN3730, Q4 DMN3730

Commit message: Optimize component base
Parts:
- C95: footprint Fabmicro:C_0402_1005Metric -> Capacitor_SMD:C_0402_1005Metric; Mfr. Part Number CL05B104K05NNNC -> CC0402KRX7R9BB104
Changed lines of the file:
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@@
   (title_block
     (title "ПИР СЦХ-254 \"Карно\"\n(Karnix ASB-254)")
-    (date "2023-10-20")
+    (date "2023-10-21")
     (rev "V1.0")
     (company "ООО \"Фабмикро\"")
@@
       (effects (font (size 1.27 1.27)) (justify left))
     )
-    (property "Footprint" "Fabmicro:C_0402_1005Metric" (at 149.8092 165.354 90)
+    (property "Footprint" "Capacitor_SMD:C_0402_1005Metric" (at 149.8092 165.354 90)
       (effects (font (size 1.27 1.27)) hide)
     )
@@
       (effects (font (size 1.27 1.27)) hide)
     )
-    (property "Mfr. Part Number" "CL05B104K05NNNC" (at 148.844 161.544 0)
+    (property "Mfr. Part Number" "CC0402KRX7R9BB104" (at 148.844 161.544 0)
       (effects (font (size 1.27 1.27)) hide)
     )
@@
       (effects (font (size 1.27 1.27)) (justify left))
     )
-    (property "Footprint" "Fabmicro:C_0402_1005Metric" (at 150.1902 139.7 90)
+    (property "Footprint" "Capacitor_SMD:C_0402_1005Metric" (at 150.1902 139.7 90)
       (effects (font (size 1.27 1.27)) hide)
     )
@@
       (effects (font (size 1.27 1.27)) hide)
     )
-    (property "Mfr. Part Number" "CL05B104K05NNNC" (at 149.225 135.89 0)
-      (effects (font (size 1.27 1.27)) hide)
-    )
+    (property "Mfr. Part Number" "CC0402KRX7R9BB104" (at 149.225 135.89 0)
+      (effects (font (size 1.27 1.27)) hide)
+    )
