File: Karnix_ASB-254-v1.0/SRAM.kicad_sch (KiCad schematic)
At the start: 4 parts, among them U21 K6R4016V1D-TC10 (TSOP-44, +3.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

Commit message: Optimize component base
Parts:
- C99: footprint Fabmicro:C_0402_1005Metric -> Capacitor_SMD:C_0402_1005Metric; Mfr. Part Number CL05B104K05NNNC -> CC0402KRX7R9BB104
Changed lines of the file:
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@@
   (title_block
     (title "ПИР СЦХ-254 \"Карно\"\n(Karnix ASB-254)")
-    (date "2023-10-20")
+    (date "2023-10-21")
     (rev "V1.0")
     (company "ООО \"Фабмикро\"")
@@
       (effects (font (size 1.27 1.27)) (justify left))
     )
-    (property "Footprint" "Fabmicro:C_0402_1005Metric" (at 208.4578 154.051 90)
+    (property "Footprint" "Capacitor_SMD:C_0402_1005Metric" (at 208.4578 154.051 90)
       (effects (font (size 1.27 1.27)) hide)
     )
@@
       (effects (font (size 1.27 1.27)) hide)
     )
-    (property "Mfr. Part Number" "CL05B104K05NNNC" (at 209.423 150.241 0)
+    (property "Mfr. Part Number" "CC0402KRX7R9BB104" (at 209.423 150.241 0)
       (effects (font (size 1.27 1.27)) hide)
     )
@@
       (effects (font (size 1.27 1.27)) (justify left))
     )
-    (property "Footprint" "Fabmicro:C_0402_1005Metric" (at 214.831 153.9848 90)
+    (property "Footprint" "Capacitor_SMD:C_0402_1005Metric" (at 214.831 153.9848 90)
       (effects (font (size 1.27 1.27)) hide)
     )
@@
       (effects (font (size 1.27 1.27)) hide)
     )
-    (property "Mfr. Part Number" "CL05B104K05NNNC" (at 215.7962 150.1748 0)
-      (effects (font (size 1.27 1.27)) hide)
-    )
+    (property "Mfr. Part Number" "CC0402KRX7R9BB104" (at 215.7962 150.1748 0)
+      (effects (font (size 1.27 1.27)) hide)
+    )
