File: Karnix_ASB-254-v1.1/FTDI_Prog.kicad_sch (KiCad schematic)
At the start: 29 parts, among them J1 USB_C_Receptacle_USB2.0, U20 FT2232D, Y1 6MHz

Commit message: Bugfixes and improvements:
1. FT2232D VCCIOA and VCCIOB connect to 3V3OUT to provide 3.3V I/O
2. Add SW5 button connected to FPGA_RESET as main reset signal
3. Length match HDMI diff pairs
Connections:
- net FT_VCC: no longer U20.14 (VCCIOA), U20.31 (VCCIOB)
- net at C99.1, U20.6 (3V3OUT): now also U20.14 (VCCIOA), U20.31 (VCCIOB)
Changed lines of the file:
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@@
   (junction (at 107.5529 121.8579) (diameter 0) (color 0 0 0 0)
   )
+  (junction (at 235.585 97.917) (diameter 0) (color 0 0 0 0)
+  )
   (junction (at 240.665 110.617) (diameter 0) (color 0 0 0 0)
   )
@@
   (junction (at 122.936 121.8579) (diameter 0) (color 0 0 0 0)
   )
-  (junction (at 240.665 87.757) (diameter 0) (color 0 0 0 0)
-  )
-  (junction (at 240.665 90.297) (diameter 0) (color 0 0 0 0)
-  )
   (junction (at 210.185 85.217) (diameter 0) (color 0 0 0 0)
   )
@@
   )
   (junction (at 304.8963 128.7282) (diameter 0) (color 0 0 0 0)
+  )
+  (junction (at 240.665 92.837) (diameter 0) (color 0 0 0 0)
   )
   (junction (at 107.5529 124.3979) (diameter 0) (color 0 0 0 0)
@@
     (stroke (width 0) (type default))
   )
+  (wire (pts (xy 240.665 92.837) (xy 235.585 92.837))
+    (stroke (width 0) (type default))
+  )
   (wire (pts (xy 291.465 151.257) (xy 296.545 151.257))
     (stroke (width 0) (type default))
@@
     (stroke (width 0) (type default))
   )
-  (wire (pts (xy 240.665 90.297) (xy 240.665 87.757))
-    (stroke (width 0) (type default))
-  )
   (wire (pts (xy 189.865 97.917) (xy 189.865 95.377))
     (stroke (width 0) (type default))
@@
     (stroke (width 0) (type default))
   )
+  (wire (pts (xy 235.585 92.837) (xy 235.585 97.917))
+    (stroke (width 0) (type default))
+  )

Commit message: Save USB type C connector footprint to local lib, add paste to through-hole pins
Parts:
- J1: footprint Connector_USB:USB_C_Receptacle_HRO_TYPE-C-31-M-12 -> Fabmicro:USB_C_Receptacle_HRO_TYPE-C-31-M-12
Changed lines of the file:
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@@
       (effects (font (size 1.27 1.27)))
     )
-    (property "Footprint" "Connector_USB:USB_C_Receptacle_HRO_TYPE-C-31-M-12" (at 93.5829 121.8579 0)
+    (property "Footprint" "Fabmicro:USB_C_Receptacle_HRO_TYPE-C-31-M-12" (at 93.5829 121.8579 0)
       (effects (font (size 1.27 1.27)) hide)
     )
