File: Karnix_ASB-254-v1.1/Karnix_ASB.kicad_sch (KiCad schematic)
At the start: 59 parts, among them J4 Conn_01x07, SW1 SW_Push, SW2 SW_Push, SW3 SW_Push, SW4 SW_Push

Commit message: Bugfixes and improvements:
1. FT2232D VCCIOA and VCCIOB connect to 3V3OUT to provide 3.3V I/O
2. Add SW5 button connected to FPGA_RESET as main reset signal
3. Length match HDMI diff pairs
Parts:
- added C6: 0.1uF/50V, Capacitor_SMD:C_0402_1005Metric, symbol Fabmicro:CapacitorUnpolarized
- added R?: 1K/1%, Fabmicro:R_0402_1005Metric, symbol Fabmicro:Resistor
- added SW5: SW_Push, Button_Switch_SMD:SW_SPST_EVQPE1, symbol Switch:SW_Push
- D1, D3: value FYLS-0603URC -> FYLS-0603PGC; Mfr. Part Number FYLS-0603URC -> FYLS-0603PGC
Connections:
- net FPGA_RESET: now also C6.1, SW5.1
- net GND: now also C6.2, R?.2
- new net: R?.1, SW5.2
Changed lines of the file:
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@@
   (junction (at 153.1304 142.24) (diameter 0) (color 0 0 0 0)
   )
+  (junction (at 168.656 173.482) (diameter 0) (color 0 0 0 0)
+  )
   (junction (at 153.035 157.607) (diameter 0) (color 0 0 0 0)
   )
+  (junction (at 131.3895 173.482) (diameter 0) (color 0 0 0 0)
+  )
   (wire (pts (xy 244.5 184.8) (xy 244.5 181.82))
     (stroke (width 0) (type default))
@@
     (stroke (width 0) (type default))
   )
+  (wire (pts (xy 124.7148 173.482) (xy 131.3895 173.482))
+    (stroke (width 0) (type default))
+  )
   (wire (pts (xy 137.287 115.316) (xy 134.747 115.316))
     (stroke (width 0) (type default))
@@
     (stroke (width 0) (type default))
   )
+  (wire (pts (xy 168.656 173.482) (xy 168.656 180.086))
+    (stroke (width 0) (type default))
+  )
   (wire (pts (xy 239.5 166.6) (xy 246.5 166.6))
     (stroke (width 0) (type default))
@@
     (stroke (width 0) (type default))
   )
+  (wire (pts (xy 131.3895 174.6287) (xy 131.3895 173.482))
+    (stroke (width 0) (type default))
+  )
   (wire (pts (xy 233.0774 97.6461) (xy 243.2374 97.6461))
     (stroke (width 0) (type default))
@@
     (stroke (width 0) (type default))
   )
-  (wire (pts (xy 168.656 171.196) (xy 168.656 164.719))
+  (wire (pts (xy 168.656 164.719) (xy 168.656 173.482))
     (stroke (width 0) (type default))
   )
@@
     (stroke (width 0) (type default))
   )
+  (wire (pts (xy 152.6548 173.482) (xy 155.067 173.482))
+    (stroke (width 0) (type default))
+  )
   (wire (pts (xy 255.9374 100.1861) (xy 266.0974 100.1861))
     (stroke (width 0) (type default))
@@
     (stroke (width 0) (type default))
   )
+  (wire (pts (xy 131.3895 173.482) (xy 142.4948 173.482))
+    (stroke (width 0) (type default))
+  )
+  (wire (pts (xy 165.227 173.482) (xy 168.656 173.482))
+    (stroke (width 0) (type default))
+  )
   (wire (pts (xy 84.836 97.155) (xy 87.376 97.155))
     (stroke (width 0) (type default))
@@
     )
   )
+  (global_label "FPGA_RESET" (shape input) (at 124.7148 173.482 180)
+    (effects (font (size 1.27 1.27)) (justify right))
+    (property "Intersheetrefs" "${INTERSHEET_REFS}" (at 124.7148 173.482 0)
+      (effects (font (size 1.27 1.27)) hide)
+    )
+  )
   (global_label "GPIO_04" (shape input) (at 212.7574 95.1061 180)
     (effects (font (size 1.27 1.27)) (justify right))
@@
       (effects (font (size 1.27 1.27)))
     )
-    (property "Value" "FYLS-0603URC" (at 156.5148 110.8886 0)
+    (property "Value" "FYLS-0603PGC" (at 156.5148 110.8886 0)
       (effects (font (size 1.27 1.27)))
     )
@@
       (effects (font (size 1.27 1.27)) hide)
     )
-    (property "Mfr. Part Number" "FYLS-0603URC" (at 160.147 107.7136 0)
+    (property "Mfr. Part Number" "FYLS-0603PGC" (at 160.147 107.7136 0)
       (effects (font (size 1.27 1.27)) hide)
     )
@@
     )
   )
+  (symbol (lib_id "power:GND") (at 131.3895 179.7087 0) (mirror y) (unit 1)
+    (in_bom yes) (on_board yes) (dnp no)
+    (property "Reference" "#PWR?" (at 131.3895 186.0587 0)
+      (effects (font (size 1.27 1.27)) hide)
+    )
+    (property "Value" "GND" (at 131.3895 183.5187 0)
+      (effects (font (size 1.27 1.27)))
+    )
+    (property "Footprint" "" (at 131.3895 179.7087 0)
+      (effects (font (size 1.27 1.27)) hide)
+    )
+    (property "Datasheet" "" (at 131.3895 179.7087 0)
+      (effects (font (size 1.27 1.27)) hide)
+    )
+    (pin "1")
+    (instances
+      (project "Karnix_ASB"
+        (path "/fe37e245-9527-4c72-91fc-09b617a42f73/00000000-0000-0000-0000-0000602e11fa"
+          (reference "#PWR?") (unit 1)
+        )
+        (path "/fe37e245-9527-4c72-91fc-09b617a42f73/00000000-0000-0000-0000-0000602e119a"
+          (reference "#PWR063") (unit 1)
+        )
+        (path "/fe37e245-9527-4c72-91fc-09b617a42f73"
+          (reference "#PWR0222") (unit 1)
+        )
+      )
+    )
+  )
   (symbol (lib_id "power:GND") (at 85.979 207.645 90) (unit 1)
     (in_bom yes) (on_board yes) (dnp no)
@@
     )
   )
+  (symbol (lib_id "Fabmicro:CapacitorUnpolarized") (at 131.3895 177.1687 270) (unit 1)
+    (in_bom yes) (on_board yes) (dnp no)
+    (property "Reference" "C6" (at 135.1995 177.1687 90)
+      (effects (font (size 1.27 1.27)) (justify left))
+    )
+    (property "Value" "0.1uF/50V" (at 132.6595 179.7087 90)
+      (effects (font (size 1.27 1.27)) (justify left))
+    )
+    (property "Footprint" "Capacitor_SMD:C_0402_1005Metric" (at 132.3547 180.9787 90)
+      (effects (font (size 1.27 1.27)) hide)
+    )
+    (property "Datasheet" "~" (at 131.3895 177.1687 90)
+      (effects (font (size 1.27 1.27)) hide)
+    )
+    (property "Mfr. Part Number" "CC0402KRX7R9BB104" (at 131.3895 177.1687 0)
+      (effects (font (size 1.27 1.27)) hide)
+    )
+    (property "Supplier" "Fabmicro" (at 131.3895 177.1687 0)
+      (effects (font (size 1.27 1.27)) hide)
+    )
+    (pin "1")
+    (pin "2")
+    (instances
+      (project "Karnix_ASB"
+        (path "/fe37e245-9527-4c72-91fc-09b617a42f73/00000000-0000-0000-0000-0000602e0fd3"
+          (reference "C6") (unit 1)
+        )
+        (path "/fe37e245-9527-4c72-91fc-09b617a42f73"
+          (reference "C92") (unit 1)
+        )
+      )
+    )
+  )
   (symbol (lib_id "Fabmicro:CONN_2Pins") (at 72.898 215.773 0) (unit 1)
     (in_bom yes) (on_board yes) (dnp no)
@@
       (effects (font (size 1.27 1.27)))
     )
-    (property "Value" "FYLS-0603URC" (at 156.5148 103.124 0)
+    (property "Value" "FYLS-0603PGC" (at 156.5148 103.124 0)
       (effects (font (size 1.27 1.27)))
     )
@@
       (effects (font (size 1.27 1.27)) hide)
     )
-    (property "Mfr. Part Number" "FYLS-0603URC" (at 160.147 99.949 0)
+    (property "Mfr. Part Number" "FYLS-0603PGC" (at 160.147 99.949 0)
+      (effects (font (size 1.27 1.27)) hide)
+    )
+    (property "Field5" "" (at 160.147 99.949 0)
       (effects (font (size 1.27 1.27)) hide)
     )
@@
     )
   )
-  (symbol (lib_id "power:GND") (at 168.656 171.196 0) (mirror y) (unit 1)
+  (symbol (lib_id "power:GND") (at 168.656 180.086 0) (mirror y) (unit 1)
     (in_bom yes) (on_board yes) (dnp no)
-    (property "Reference" "#PWR?" (at 168.656 177.546 0)
+    (property "Reference" "#PWR?" (at 168.656 186.436 0)
       (effects (font (size 1.27 1.27)) hide)
     )
-    (property "Value" "GND" (at 168.656 175.006 0)
+    (property "Value" "GND" (at 168.656 183.896 0)
       (effects (font (size 1.27 1.27)))
     )
-    (property "Footprint" "" (at 168.656 171.196 0)
+    (property "Footprint" "" (at 168.656 180.086 0)
       (effects (font (size 1.27 1.27)) hide)
     )
-    (property "Datasheet" "" (at 168.656 171.196 0)
+    (property "Datasheet" "" (at 168.656 180.086 0)
       (effects (font (size 1.27 1.27)) hide)
     )
@@
     )
   )
+  (symbol (lib_id "Switch:SW_Push") (at 147.5748 173.482 0) (unit 1)
+    (in_bom yes) (on_board yes) (dnp no)
+    (property "Reference" "SW5" (at 135.3828 172.1677 0)
+      (effects (font (size 1.27 1.27)))
+    )
+    (property "Value" "SW_Push" (at 141.3518 172.1677 0)
+      (effects (font (size 1.27 1.27)))
+    )
+    (property "Footprint" "Button_Switch_SMD:SW_SPST_EVQPE1" (at 147.5748 168.402 0)
+      (effects (font (size 1.27 1.27)) hide)
+    )
+    (property "Datasheet" "~" (at 147.5748 168.402 0)
+      (effects (font (size 1.27 1.27)) hide)
+    )
+    (property "Mfr. Part Number" "DTSM-32" (at 147.5748 173.482 0)
+      (effects (font (size 1.27 1.27)) hide)
+    )
+    (pin "1")
+    (pin "2")
+    (instances
+      (project "Karnix_ASB"
+        (path "/fe37e245-9527-4c72-91fc-09b617a42f73"
+          (reference "SW5") (unit 1)
+        )
+      )
+    )
+  )
   (symbol (lib_id "Connector_Generic:Conn_02x20_Odd_Even") (at 248.3174 110.3461 0) (unit 1)
     (in_bom yes) (on_board yes) (dnp no) (fields_autoplaced)
@@
       (effects (font (size 1.27 1.27)))
     )
-    (property "Value" "FYLS-0603URC" (at 156.5148 118.491 0)
+    (property "Value" "FYLS-0603PGC" (at 156.5148 118.491 0)
       (effects (font (size 1.27 1.27)))
     )
@@
       (effects (font (size 1.27 1.27)) hide)
     )
-    (property "Mfr. Part Number" "FYLS-0603URC" (at 160.147 115.316 0)
+    (property "Mfr. Part Number" "FYLS-0603PGC" (at 160.147 115.316 0)
       (effects (font (size 1.27 1.27)) hide)
     )
@@
         )
       )
+    )
+  )
+  (symbol (lib_id "Fabmicro:Resistor") (at 160.147 173.482 0) (unit 1)
+    (in_bom yes) (on_board yes) (dnp no)
+    (property "Reference" "R?" (at 156.337 171.704 0)
+      (effects (font (size 1.27 1.27)) (justify left))
+    )
+    (property "Value" "1K/1%" (at 159.893 171.577 0)
+      (effects (font (size 1.27 1.27)) (justify left))
+    )
+    (property "Footprint" "Fabmicro:R_0402_1005Metric" (at 160.147 175.26 0)
+      (effects (font (size 1.27 1.27)) hide)
+    )
+    (property "Datasheet" "" (at 160.147 173.482 90)
+      (effects (font (size 1.27 1.27)) hide)
+    )
+    (property "Mfr. Part Number" "RC0402FR-071KL" (at 160.147 173.482 0)
+      (effects (font (size 1.27 1.27)) hide)
+    )
+    (property "Supplier" "" (at 160.147 173.482 0)
+      (effects (font (size 1.27 1.27)) hide)
+    )
+    (pin "1")
+    (pin "2")
+    (instances
+      (project "Karnix_ASB"
+        (path "/fe37e245-9527-4c72-91fc-09b617a42f73/00000000-0000-0000-0000-0000602e11fa"
+          (reference "R?") (unit 1)
+        )
+        (path "/fe37e245-9527-4c72-91fc-09b617a42f73/00000000-0000-0000-0000-0000602e119a"
+          (reference "R11") (unit 1)
+        )
+        (path "/fe37e245-9527-4c72-91fc-09b617a42f73"
+          (reference "R168") (unit 1)
+        )
+      )

Commit message: Change GPIO current limiting resistors form 110R to 51R. Update modification date.
Parts:
- R32, R33, R34, R35, R36, R37, R38, R39, R42, R43, R44, R45, R46, R47, R48, R49: value 110R/1% -> 51R/1%; Mfr. Part Number RC0402FR-07110RL -> RC0402FR-0751RL
