File: Karnix_ASB-254-v1.1/SRAM.kicad_sch (KiCad schematic)
At the start: 4 parts, among them U21 K6R4016V1D-TC10 (TSOP-44, +3.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

Commit message: U21: remove comma character in value field, which is causing problems with assembly
Parts:
- U21: value K6R4016V1D-TC10 (TSOP-44, +3.3V) -> K6R4016V1D-TC10 (TSOP-44/+3.3V)
Changed lines of the file:
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@@
       (effects (font (size 1.27 1.27)))
     )
-    (property "Value" "K6R4016V1D-TC10 (TSOP-44, +3.3V)" (at 182.753 88.635 0)
+    (property "Value" "K6R4016V1D-TC10 (TSOP-44/+3.3V)" (at 182.753 88.635 0)
       (effects (font (size 1.27 1.27)))
     )
